Commit message: Updated the urdf model

File: dwl/sample/hyq.urdf (robot description, URDF)
Before this commit: robot hyq, 18 links, 17 joints
Links:
- link lf_foot: geometry collision sphere radius=0.02175; visual sphere radius=0.02175
- link lh_foot: geometry collision sphere radius=0.02175; visual sphere radius=0.02175
- link rf_foot: geometry collision sphere radius=0.02175; visual sphere radius=0.02175
- link rh_foot: geometry collision sphere radius=0.02175; visual sphere radius=0.02175
- link trunk: mass 71.758 -> 59.1
Joints:
- joint lf_foot_joint: origin xyz=0.341 0 0 rpy=1.57079632679 0 -1.57079632679 -> xyz=0.346 0 0 rpy=1.57079632679 0 -1.57079632679
- joint lh_foot_joint: origin xyz=0.341 0 0 rpy=1.57079632679 0 -1.57079632679 -> xyz=0.346 0 0 rpy=1.57079632679 0 -1.57079632679
- joint rf_foot_joint: origin xyz=0.341 0 0 rpy=1.57079632679 0 -1.57079632679 -> xyz=0.346 0 0 rpy=1.57079632679 0 -1.57079632679
- joint rh_foot_joint: origin xyz=0.341 0 0 rpy=1.57079632679 0 -1.57079632679 -> xyz=0.346 0 0 rpy=1.57079632679 0 -1.57079632679
